Commit message: add ros2_control unity hardware

File: zx120_description/urdf/zx120.xacro (robot description, xacro)
@@ -5,4 +5,5 @@
 	<!-- Import Rviz colors -->
 	<!-- <xacro:include filename="$(find zx120_description)/urdf/materials.xacro" /> -->
+  <!-- <xacro:include filename="$(find zx120_description)/urdf/zx120.ros2_control.xacro" /> -->
 	<!-- Base Link -->
 	<link name="base_link"/>
@@ -151,5 +152,5 @@
         <box size="0.001 0.001 0.001" />
       </geometry>
-      <material name="red"/>
+      <!-- <material name="red"/> -->
     </visual>
     <inertial>
@@ -168,53 +169,4 @@
     <limit effort="1" lower="-3.14" upper="3.14" velocity="0.5"/>
   </joint>
-	<transmission name="tran1">
-		<type>transmission_interface/SimpleTransmission</type>
-		<joint name="swing_joint">
-			<hardwareInterface>hardware_interface/PositionJointInterface</hardwareInterface>
-		</joint>
-		<actuator name="motor1">
-			<hardwareInterface>hardware_interface/PositionJointInterface</hardwareInterface>
-			<mechanicalReduction>1</mechanicalReduction>
-		</actuator>
-	</transmission>
-	<transmission name="tran2">
-		<type>transmission_interface/SimpleTransmission</type>
-		<joint name="boom_joint">
-			<hardwareInterface>hardware_interface/PositionJointInterface</hardwareInterface>
-		</joint>
-		<actuator name="motor2">
-			<hardwareInterface>hardware_interface/PositionJointInterface</hardwareInterface>
-			<mechanicalReduction>1</mechanicalReduction>
-		</actuator>
-	</transmission>
-	<transmission name="tran3">
-		<type>transmission_interface/SimpleTransmission</type>
-		<joint name="arm_joint">
-			<hardwareInterface>hardware_interface/PositionJointInterface</hardwareInterface>
-		</joint>
-		<actuator name="motor3">
-			<hardwareInterface>hardware_interface/PositionJointInterface</hardwareInterface>
-			<mechanicalReduction>1</mechanicalReduction>
-		</actuator>
-	</transmission>
-	<transmission name="tran4">
-		<type>transmission_interface/SimpleTransmission</type>
-		<joint name="bucket_joint">
-			<hardwareInterface>hardware_interface/PositionJointInterface</hardwareInterface>
-		</joint>
-		<actuator name="motor4">
-			<hardwareInterface>hardware_interface/PositionJointInterface</hardwareInterface>
-			<mechanicalReduction>1</mechanicalReduction>
-		</actuator>
-	</transmission>
-  <transmission name="dummy_trans1">
-    <type>transmission_interface/SimpleTransmission</type>
-      <joint name="bucket_end_joint">
-      <hardwareInterface>hardware_interface/PositionJointInterface</hardwareInterface>
-    </joint>
-    <actuator name="dummy_motor1">
-      <hardwareInterface>hardware_interface/PositionJointInterface</hardwareInterface>
-      <mechanicalReduction>1</mechanicalReduction>
-    </actuator>
-  </transmission>
+	<!-- <xacro:zx120_ros2_control/> -->
 </robot>

File: zx120_moveit_config/config/zx120.ros2_control.xacro (robot description, xacro)
@@ -1,5 +1,5 @@
 <?xml version="1.0"?>
 <robot xmlns:xacro="http://www.ros.org/wiki/xacro">
-    <xacro:macro name="zx120_ros2_control" params="name initial_positions_file">
+    <xacro:macro name="zx120_ros2_control" params="name plugin initial_positions_file">
         <xacro:property name="initial_positions" value="${load_yaml(initial_positions_file)['initial_positions']}"/>
         <ros2_control name="${name}" type="system">
@@ -7,5 +7,5 @@
                 <!-- By default, set up controllers for simulation. This won't work on real hardware -->
                 <!-- <plugin>mock_components/GenericSystem</plugin> -->
-                <plugin>zx120_control_hardware/Zx120UpperArmPositionHardware</plugin>
+                <plugin>${plugin}</plugin>
             </hardware>
             <joint name="swing_joint">

File: zx120_moveit_config/config/zx120_unity.urdf.xacro (robot description, xacro)
@@ -8,5 +8,5 @@
     <!-- <xacro:include filename="$(find zx120_moveit_config)/config/zx120.ros2_control.xacro" /> -->
     <!-- <xacro:zx120_ros2_control name="FakeSystem" initial_positions_file="$(arg initial_positions_file)"/> -->
-    <xacro:zx120_ros2_control name="trajectory_control" plugin="zx120_control_hardware/Zx120UpperArmPositionHardware" initial_positions_file="$(arg initial_positions_file)"/>
+    <xacro:zx120_ros2_control name="trajectory_control" plugin="zx120_control_hardware/Zx120UpperArmPositionUnityHardware" initial_positions_file="$(arg initial_positions_file)"/>
     <!-- The name must not be ideal(not same as Zx120UpperArmPositionHardware) -->
 </robot>

Commit message: Fix to add namespace "zx120"

File: zx120_description/urdf/zx120.xacro (robot description, xacro)
@@ -7,11 +7,11 @@
   <!-- <xacro:include filename="$(find zx120_description)/urdf/zx120.ros2_control.xacro" /> -->
 	<!-- Base Link -->
-	<link name="base_link"/>
-	<joint name="base_joint" type="fixed">
-		<parent link="base_link"/>
-		<child link="track_link"/>
+	<link name="zx120/base_link"/>
+	<joint name="zx120/base_joint" type="fixed">
+		<parent link="zx120/base_link"/>
+		<child link="zx120/track_link"/>
 	</joint>
 	<!-- Base Link -->
-	<link name="track_link">
+	<link name="zx120/track_link">
 		<visual>
 			<geometry>
@@ -33,11 +33,11 @@
 	</link>
 	<!-- body axis -->
-	<joint name="swing_joint" type="continuous">
+	<joint name="zx120/swing_joint" type="continuous">
 		<origin xyz="0 0 1"/>
 		<axis xyz="0 0 2"/>
-		<parent link="track_link"/>
-		<child link="body_link"/>
+		<parent link="zx120/track_link"/>
+		<child link="zx120/body_link"/>
 	</joint>
-	<link name="body_link">
+	<link name="zx120/body_link">
 		<visual>
 			<origin xyz="0 0 0"/>
@@ -61,12 +61,12 @@
 	</link>
 	<!-- boom axis -->
-	<joint name="boom_joint" type="revolute">
+	<joint name="zx120/boom_joint" type="revolute">
 		<origin xyz="0.14 -0.16443 0.424" rpy="0 ${radians(90)} 0"/>
 		<axis xyz="0 1 0"/>
-		<parent link="body_link"/>
-		<child link="boom_link"/>
+		<parent link="zx120/body_link"/>
+		<child link="zx120/boom_link"/>
 		<limit lower="${radians(-70)}" upper="${radians(44)}" effort="500" velocity="6.159937255"/>
 	</joint>
-	<link name="boom_link">
+	<link name="zx120/boom_link">
 		<visual>
 			<origin xyz="0 0 0" rpy="0 -1.185 0"/>
@@ -89,12 +89,12 @@
 		</inertial>
 	</link>
-	<joint name="arm_joint" type="revolute">
+	<joint name="zx120/arm_joint" type="revolute">
 		<origin xyz="0 0 4.6"/>
 		<axis xyz="0 1 0"/>
-		<parent link="boom_link"/>
-		<child link="arm_link"/>
+		<parent link="zx120/boom_link"/>
+		<child link="zx120/arm_link"/>
 	    <limit effort="1" lower="${radians(30)}" upper="${radians(152)}" velocity="0.5"/>
 	</joint>
-	<link name="arm_link">
+	<link name="zx120/arm_link">
 		<visual>
 			<origin xyz="0 0 0" rpy="0 3.28 0"/>
@@ -118,12 +118,12 @@
 	</link>
 	<!-- bucket axis -->
-	<joint name="bucket_joint" type="revolute">
+	<joint name="zx120/bucket_joint" type="revolute">
 		<origin xyz="0 0 2.519"/>
 		<axis xyz="0 1 0"/>
-		<parent link="arm_link"/>
-		<child link="bucket_link"/>
+		<parent link="zx120/arm_link"/>
+		<child link="zx120/bucket_link"/>
 	    <limit effort="1" lower="${radians(-33)}" upper="${radians(143)}" velocity="0.5"/>
 	</joint>
-	<link name="bucket_link">
+	<link name="zx120/bucket_link">
 		<visual>
 			<origin xyz="0 0 0" rpy="0 0.75 0"/>
@@ -146,5 +146,5 @@
 		</inertial>
 	</link>
-  <link name="bucket_end_link">
+  <link name="zx120/bucket_end_link">
     <visual>
       <origin xyz="0 0 0" rpy="0 0 0"/>
@@ -162,7 +162,7 @@
     </inertial>
   </link>
-  <joint name="bucket_end_joint" type="revolute">
-    <parent link="bucket_link"/>
-    <child link="bucket_end_link"/>
+  <joint name="zx120/bucket_end_joint" type="revolute">
+    <parent link="zx120/bucket_link"/>
+    <child link="zx120/bucket_end_link"/>
     <axis xyz="1 0 0"/>
     <origin rpy="0 ${radians(50)} 0" xyz="0 0 1.23"/>
